File: hardware/minipid.sch (KiCad schematic (older format))
At the start: 24 parts, among them J1 Mains, J2 Load, J3 PT1000, J4 ISP, J5 Display, J6 UART, U1 ATtiny45-20PU, U2 LP2950-5.0_TO92, U3 MOC3063M

Commit message: hardware: fix Triac name
Signed-off-by: Michael Walle <michael@walle.cc>
Parts:
- D2: value BTA 08/600BW -> BTA 08/600CW; Reichelt BTB 08/600BW -> BTA 08/600CW
Changed lines of the file:
@@
 P 1700 2950
 F 0 "D2" H 1750 3050 50  0000 L CNN
-F 1 "BTA 08/600BW" H 1050 2750 50  0000 L CNN
+F 1 "BTA 08/600CW" H 1050 2750 50  0000 L CNN
 F 2 "Package_TO_SOT_THT:TO-220-3_Horizontal_TabDown" V 1775 2975 50  0001 C CNN
 F 3 "~" V 1700 2950 50  0001 C CNN
-F 4 "BTB 08/600BW" H 0   0   50  0001 C CNN "Reichelt"
+F 4 "BTA 08/600CW" H 0   0   50  0001 C CNN "Reichelt"
 	1    1700 2950
 	-1   0    0    -1
